Commit message: corect transformation of saving

File: urdf/robotic_cell.urdf.xacro (robot description, xacro)
@@ -25,5 +25,6 @@
   <!-- ACTUAL PROGRAM-->
   <xacro:property name="parrent_package_name" value="rviz_plugin_urdf_composer" />
-  <xacro:property name="yaml_file" value="$(find ${parrent_package_name})/config/active_config.yaml" />
+  <xacro:arg name="yaml_name"  default="active_config"/>
+  <xacro:property name="yaml_file" value="$(find ${parrent_package_name})/config/$(arg yaml_name).yaml" />
   <xacro:property name="active_config" value="${xacro.load_yaml(yaml_file)}"/>
   <xacro:property name="list_of_active_elements_names" value="${active_config['active_description_elements']}"/>

Commit message: loading config yamls

File: urdf/robotic_cell.urdf.xacro (robot description, xacro)
@@ -26,5 +26,10 @@
   <xacro:property name="parrent_package_name" value="rviz_plugin_urdf_composer" />
   <xacro:arg name="yaml_name"  default="active_config"/>
+  <xacro:arg name="yaml_path"  default="none"/>
+  <xacro:property name="yaml_path_property"  value="$(arg yaml_path)"/>
   <xacro:property name="yaml_file" value="$(find ${parrent_package_name})/config/$(arg yaml_name).yaml" />
+  <xacro:if value="${yaml_path_property != 'none'}">
+    <xacro:property name="yaml_file" value="${yaml_path_property}" />
+  </xacro:if>
   <xacro:property name="active_config" value="${xacro.load_yaml(yaml_file)}"/>
   <xacro:property name="list_of_active_elements_names" value="${active_config['active_description_elements']}"/>
